File: eagle-pcb/boardv2.brd (EAGLE design)
At the start: 39.4 x 12 mm, 11 parts, among them IC1 ATTINY85, J1 FEMALE 2x3, X1 USBPCB

Commit message: FIX pcb, use MOSI to drive LED, not RESET
Parts:
- moved J1 2.79 mm to (34.4, 7.11)
- moved D3 1.27 mm to (26.7, 9.50)
- moved D4 1.27 mm to (26.7, 9.50)
Connections:
- removed net RESET/LED: D3.4, IC1.1, J1.6
- new net RESET: IC1.1, J1.5
- net MISO: now also D3.4, J1.6; no longer J1.5
Routing:
- net RESET/LED: track 18.5 -> 0.00 mm
- net RESET: track 0.00 -> 16.5 mm
- net MISO: track 25.7 -> 21.2 mm, vias 1 -> 2
- net SDA/MOSI: track 28.5 -> 25.7 mm
- net SCK: track 18.1 -> 15.4 mm
- net 5V: track 54.3 -> 51.7 mm
- net N$2: track 3.07 -> 2.35 mm
Other:
- board size 39.4 x 12 mm -> 36.6 x 12 mm
